File: KiCad/RP2040-MiniPill-Breakout-Board.kicad_pcb (KiCad board)
At the start: 2 copper layers, 52 x 66.5 mm, 27 parts, among them J1 Conn_01x20_Socket, J2 Conn_01x20_Socket, J3 Screw_Terminal_01x20, J4 Screw_Terminal_01x20, Q1 IRLML6402, Q2 IRLML2502, U1 TPS3700

Commit message: changing UV
Parts:
- C1: value C -> 100n
- R2: value 100 -> 56
Changed lines of the file:
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@@
 			)
 		)
+		(property "LCSC" "C915914 (4x)"
+			(at 0 0 270)
+			(unlocked yes)
+			(layer "F.Fab")
+			(hide yes)
+			(effects
+				(font
+					(size 1 1)
+					(thickness 0.15)
+				)
+			)
+		)
 		(property ki_fp_filters "TerminalBlock*:*")
 		(sheetname "/")
 		(sheetfile "RP2040-MiniPill-Breakout-Board.kicad_sch")
-		(attr through_hole)
+		(attr through_hole exclude_from_pos_files)
 		(fp_line
 			(start -1.64 3.52)
@@
 			)
 		)
+		(property "LCSC" "C861451"
+			(at 0 0 0)
+			(unlocked yes)
+			(layer "F.Fab")
+			(hide yes)
+			(effects
+				(font
+					(size 1 1)
+					(thickness 0.15)
+				)
+			)
+		)
 		(property ki_fp_filters "R_*")
 		(sheetname "/")
 		(sheetfile "RP2040-MiniPill-Breakout-Board.kicad_sch")
-		(attr smd)
+		(attr smd exclude_from_pos_files)
 		(fp_line
 			(start -0.254724 -0.5225)
@@
 			)
 		)
+		(property "LCSC" "C223608"
+			(at 0 0 0)
+			(unlocked yes)
+			(layer "F.Fab")
+			(hide yes)
+			(effects
+				(font
+					(size 1 1)
+					(thickness 0.15)
+				)
+			)
+		)
 		(property ki_fp_filters "TO-???* *_Diode_* *SingleDiode* D_*")
 		(sheetname "/")
 		(sheetfile "RP2040-MiniPill-Breakout-Board.kicad_sch")
-		(attr smd)
+		(attr smd exclude_from_pos_files)
 		(fp_line
 			(start -2.21 -1)
@@
 			)
 		)
+		(property "LCSC" "C861451"
+			(at 0 0 90)
+			(unlocked yes)
+			(layer "F.Fab")
+			(hide yes)
+			(effects
+				(font
+					(size 1 1)
+					(thickness 0.15)
+				)
+			)
+		)
 		(property ki_fp_filters "R_*")
 		(sheetname "/")
 		(sheetfile "RP2040-MiniPill-Breakout-Board.kicad_sch")
-		(attr smd)
+		(attr smd exclude_from_pos_files)
 		(fp_line
 			(start -0.254724 -0.5225)
@@
 			)
 		)
+		(property "LCSC" "C2589"
+			(at 0 0 90)
+			(unlocked yes)
+			(layer "F.Fab")
+			(hide yes)
+			(effects
+				(font
+					(size 1 1)
+					(thickness 0.15)
+				)
+			)
+		)
 		(property ki_fp_filters "SOT?23*")
 		(sheetname "/")
 		(sheetfile "RP2040-MiniPill-Breakout-Board.kicad_sch")
-		(attr smd)
+		(attr smd exclude_from_pos_files)
 		(fp_line
 			(start 0.76 -1.56)
@@
 			)
 		)
+		(property "LCSC" "C861451"
+			(at 0 0 0)
+			(unlocked yes)
+			(layer "F.Fab")
+			(hide yes)
+			(effects
+				(font
+					(size 1 1)
+					(thickness 0.15)
+				)
+			)
+		)
 		(property ki_fp_filters "R_*")
 		(sheetname "/")
 		(sheetfile "RP2040-MiniPill-Breakout-Board.kicad_sch")
-		(attr smd)
+		(attr smd exclude_from_pos_files)
 		(fp_line
 			(start -0.254724 -0.5225)
@@
 			)
 		)
+		(property "LCSC" "C915914 (4x)"
+			(at 0 0 270)
+			(unlocked yes)
+			(layer "F.Fab")
+			(hide yes)
+			(effects
+				(font
+					(size 1 1)
+					(thickness 0.15)
+				)
+			)
+		)
 		(property ki_fp_filters "TerminalBlock*:*")
 		(sheetname "/")
 		(sheetfile "RP2040-MiniPill-Breakout-Board.kicad_sch")
-		(attr through_hole)
+		(attr through_hole exclude_from_pos_files)
 		(fp_line
 			(start -1.64 3.52)
@@
 			)
 		)
+		(property "LCSC" "C22975"
+			(at 0 0 0)
+			(unlocked yes)
+			(layer "F.Fab")
+			(hide yes)
+			(effects
+				(font
+					(size 1 1)
+					(thickness 0.15)
+				)
+			)
+		)
 		(property ki_fp_filters "R_*")
 		(sheetname "/")
 		(sheetfile "RP2040-MiniPill-Breakout-Board.kicad_sch")
-		(attr smd)
+		(attr smd exclude_from_pos_files)
 		(fp_line
 			(start -0.254724 -0.5225)
@@
 			)
 		)
-		(property "Value" "100"
+		(property "Value" "56"
 			(at 0 1.43 90)
 			(layer "F.Fab")
@@
 			)
 		)
+		(property "LCSC" "C22775"
+			(at 0 0 270)
+			(unlocked yes)
+			(layer "F.Fab")
+			(hide yes)
+			(effects
+				(font
+					(size 1 1)
+					(thickness 0.15)
+				)
+			)
+		)
 		(property ki_fp_filters "R_*")
 		(sheetname "/")
 		(sheetfile "RP2040-MiniPill-Breakout-Board.kicad_sch")
-		(attr smd)
+		(attr smd exclude_from_pos_files)
 		(fp_line
 			(start -0.254724 0.5225)
@@
 		(sheetname "/")
 		(sheetfile "RP2040-MiniPill-Breakout-Board.kicad_sch")
-		(attr through_hole)
+		(attr through_hole exclude_from_pos_files)
 		(fp_line
 			(start -1.33 1.27)
@@
 			)
 		)
-		(property "Value" "C"
+		(property "Value" "100n"
 			(at 0 1.43 0)
 			(layer "F.Fab")
@@
 			)
 		)
+		(property "LCSC" "C14663"
+			(at 0 0 0)
+			(unlocked yes)
+			(layer "F.Fab")
+			(hide yes)
+			(effects
+				(font
+					(size 1 1)
+					(thickness 0.15)
+				)
+			)
+		)
 		(property ki_fp_filters "C_*")
 		(sheetname "/")
 		(sheetfile "RP2040-MiniPill-Breakout-Board.kicad_sch")
-		(attr smd)
+		(attr smd exclude_from_pos_files)
 		(fp_line
 			(start -0.146267 -0.51)
@@
 		(sheetname "/")
 		(sheetfile "RP2040-MiniPill-Breakout-Board.kicad_sch")
-		(attr through_hole)
+		(attr through_hole exclude_from_pos_files)
 		(fp_line
 			(start -1.33 1.27)
@@
 			)
 		)
+		(property "LCSC" "C2593"
+			(at 0 0 180)
+			(unlocked yes)
+			(layer "F.Fab")
+			(hide yes)
+			(effects
+				(font
+					(size 1 1)
+					(thickness 0.15)
+				)
+			)
+		)
 		(property ki_fp_filters "SOT?23*")
 		(sheetname "/")
 		(sheetfile "RP2040-MiniPill-Breakout-Board.kicad_sch")
-		(attr smd)
+		(attr smd exclude_from_pos_files)
 		(fp_line
 			(start 0.76 1.56)
@@
 			)
 		)
+		(property "LCSC" "C22962"
+			(at 0 0 270)
+			(unlocked yes)
+			(layer "F.Fab")
+			(hide yes)
+			(effects
+				(font
+					(size 1 1)
+					(thickness 0.15)
+				)
+			)
+		)
 		(property ki_fp_filters "R_*")
 		(sheetname "/")
 		(sheetfile "RP2040-MiniPill-Breakout-Board.kicad_sch")
-		(attr smd)
+		(attr smd exclude_from_pos_files)
 		(fp_line
 			(start -0.254724 0.5225)
@@
 			)
 		)
-		(property "Sim.Library" "Libraries/spice/TPS3700_TRANS_SIMPL.LIB"
-			(at 0 0 270)
-			(unlocked yes)
-			(layer "F.Fab")
-			(hide yes)
-			(effects
-				(font
-					(size 1 1)
-					(thickness 0.15)
-				)
-			)
-		)
-		(property "Sim.Name" "TPS3700_SIMPL"
-			(at 0 0 270)
-			(unlocked yes)
-			(layer "F.Fab")
-			(hide yes)
-			(effects
-				(font
-					(size 1 1)
-					(thickness 0.15)
-				)
-			)
-		)
-		(property "Sim.Device" "SUBCKT"
-			(at 0 0 270)
-			(unlocked yes)
-			(layer "F.Fab")
-			(hide yes)
-			(effects
-				(font
-					(size 1 1)
-					(thickness 0.15)
-				)
-			)
-		)
-		(property "Sim.Pins" "1=OUTA 2=GND 3=INA 4=INB 5=VDD 6=OUTB"
+		(property "LCSC" "C33002"
 			(at 0 0 270)
 			(unlocked yes)
@@
 		(sheetname "/")
 		(sheetfile "RP2040-MiniPill-Breakout-Board.kicad_sch")
-		(attr smd)
+		(attr smd exclude_from_pos_files)
 		(fp_line
 			(start 0 1.56)
@@
 			)
 		)
+		(property "LCSC" "C5290181"
+			(at 0 0 90)
+			(unlocked yes)
+			(layer "B.Fab")
+			(hide yes)
+			(effects
+				(font
+					(size 1 1)
+					(thickness 0.15)
+				)
+				(justify mirror)
+			)
+		)
 		(sheetname "/")
 		(sheetfile "RP2040-MiniPill-Breakout-Board.kicad_sch")
-		(attr through_hole)
+		(attr through_hole exclude_from_pos_files)
 		(fp_line
 			(start 54.62 -8.565)
@@
 			(keep_text_aligned yes)
 		)
-		(gr_text "56"
+		(gr_text "2204.7244"
 			(at 144.2 141.15 0)
 			(layer "Cmts.User")
@@
 			(keep_text_aligned yes)
 		)
-		(gr_text "4.75"
+		(gr_text "187.0079"
 			(at 137.55 63.825 90)
 			(layer "Cmts.User")
@@
 			(keep_text_aligned yes)
 		)
-		(gr_text "43.5"
+		(gr_text "1712.5984"
 			(at 144.2 135.65 0)
 			(layer "Cmts.User")
@@
 			(keep_text_aligned yes)
 		)
-		(gr_text "58"
+		(gr_text "2283.4646"
 			(at 178.05 94.7 90)
 			(layer "Cmts.User")
@@
 			(keep_text_aligned yes)
 		)
-		(gr_text "72"
+		(gr_text "2834.6457"
 			(at 185.15 94.7 90)
 			(layer "Cmts.User")
@@
 			(keep_text_aligned yes)
 		)
-		(gr_text "4.765"
+		(gr_text "187.5984"
 			(at 138.55 120.5675 90)
 			(layer "Cmts.User")
@@
 			(keep_text_aligned yes)
 		)
-		(gr_text "22.86"
+		(gr_text "900"
 			(at 144.2 54.1 0)
 			(layer "Cmts.User")
