File: KiCad/RP2040-MiniPill-Breakout-Board.kicad_sch (KiCad schematic)
At the start: 17 parts, among them J1 Conn_01x20_Socket, J2 Conn_01x20_Socket, J3 Screw_Terminal_01x20, J4 Screw_Terminal_01x20, Q1 IRLML6402, Q2 IRLML2502, U1 TPS3700

Commit message: changing UV
Parts:
- R2: value 100 -> 56
Changed lines of the file:
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@@
 			)
 		)
-		(property "Value" "100"
+		(property "Value" "56"
 			(at 57.404 102.108 0)
 			(effects
